File: Board V4/DecodingBoard/untitled.kicad_sch (KiCad schematic)
At the start: 5 parts, among them J11 CONMHF1-SMD-G-T

Commit message: Addition of the BLE module and BOM
Parts:
- removed C1: 6.63pF, symbol Device:C
- removed C2: 9.97pF, symbol Device:C
- removed FL1: DLF162500LT-5028A1, DLF162500LT-5028A1:DLF162500LT5028A1, symbol DLF162500LT-5028A1:DLF162500LT-5028A1
- removed J11: CONMHF1-SMD-G-T, CONMHF1-SMD-G-T:CONMHF1SMDGT, symbol CONMHF1-SMD-G-T:CONMHF1-SMD-G-T
- removed L1: 1.09nH, symbol Device:L
Other:
- note removed: "Low-pass filter (2.4 GHz - 2.5 GHz)"
- note removed: "Pi-network for 50 Ohm matching"
- note removed: "U.FL connector for external antenna"
- company: N-Pulse -> (none)
- title: RF circuitry & antennas -> (none)
