File: Board V4/DecodingBoard/BLE Module.kicad_sch (KiCad schematic)
At the start: 7 parts, among them IC2 RN4871-V_RM140, IC3 MCP111-195I_TO

Commit message: footprints updates
Parts:
- IC2: footprint RN4871VRM140 -> Footprints:RN4871VRM140
- IC3: footprint LR645N3GP013 -> Footprints:LR645N3GP013
Changed lines of the file:
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@@
 			)
 		)
-		(property "Footprint" "LR645N3GP013"
+		(property "Footprint" "Footprints:LR645N3GP013"
 			(at 137.16 131.75 0)
 			(hide yes)
@@
 			)
 		)
-		(property "Footprint" "RN4871VRM140"
+		(property "Footprint" "Footprints:RN4871VRM140"
 			(at 81.28 149.53 0)
 			(hide yes)
