File: Board V4/DecodingBoard/usb-c_circuit.kicad_sch (KiCad schematic)
At the start: 5 parts, among them J3 USB_C_Receptacle_USB2.0_16P, U3 USBLC6-2SC6

Commit message: Addition of the BLE module and BOM
Parts:
- removed CBUS1: 100nF, Package_TO_SOT_SMD:SOT-23-6, symbol Device:C
- added C31: 100nF, Capacitor_SMD:C_0402_1005Metric, symbol Device:C
- J3: footprint (none) -> UJ20-C-H-G-SMT-1-P16-TR
- R5, R6: footprint (none) -> Resistor_SMD:R_0402_1005Metric
Connections:
- net GND: now also C31.2
- net VBUS: now also C31.1
Changed lines of the file:
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@@
 	(title_block
 		(title "USB-C circuit")
-		(date "2026-09-29")
+		(date "2026-10-05")
 		(company "N-Pulse")
 		(comment 1 "Perrine Beurier")
@@
 			)
 		)
-		(property "Footprint" ""
+		(property "Footprint" "UJ20-C-H-G-SMT-1-P16-TR"
 			(at 44.45 46.99 0)
 			(hide yes)
@@
 				(path "/b438bce8-ca67-4245-91ae-f4475acc63f6/f85c4218-0aef-4639-a0dc-11a66bf7298f"
 					(reference "J3")
+					(unit 1)
+				)
+			)
+		)
+	)
+	(symbol
+		(lib_id "Device:C")
+		(at 107.95 31.75 90)
+		(unit 1)
+		(body_style 1)
+		(exclude_from_sim no)
+		(in_bom yes)
+		(on_board yes)
+		(in_pos_files yes)
+		(dnp no)
+		(fields_autoplaced yes)
+		(property "Reference" "C31"
+			(at 107.95 24.13 90)
+			(show_name no)
+			(do_not_autoplace no)
+			(effects
+				(font
+					(size 1.27 1.27)
+				)
+			)
+		)
+		(property "Value" "100nF"
+			(at 107.95 26.67 90)
+			(show_name no)
+			(do_not_autoplace no)
+			(effects
+				(font
+					(size 1.27 1.27)
+				)
+			)
+		)
+		(property "Footprint" "Capacitor_SMD:C_0402_1005Metric"
+			(at 111.76 30.7848 0)
+			(hide yes)
+			(show_name no)
+			(do_not_autoplace no)
+			(effects
+				(font
+					(size 1.27 1.27)
+				)
+			)
+		)
+		(property "Datasheet" ""
+			(at 107.95 31.75 0)
+			(hide yes)
+			(show_name no)
+			(do_not_autoplace no)
+			(effects
+				(font
+					(size 1.27 1.27)
+				)
+			)
+		)
+		(property "Description" "Unpolarized capacitor"
+			(at 107.95 31.75 0)
+			(hide yes)
+			(show_name no)
+			(do_not_autoplace no)
+			(effects
+				(font
+					(size 1.27 1.27)
+				)
+			)
+		)
+		(pin "2"
+		)
+		(pin "1"
+		)
+		(instances
+			(project "DecodingBoard"
+				(path "/b438bce8-ca67-4245-91ae-f4475acc63f6/f85c4218-0aef-4639-a0dc-11a66bf7298f"
+					(reference "C31")
 					(unit 1)
 				)
@@
 			)
 		)
-		(property "Footprint" ""
+		(property "Footprint" "Resistor_SMD:R_0402_1005Metric"
 			(at 73.66 41.148 90)
 			(hide yes)
@@
 				(path "/b438bce8-ca67-4245-91ae-f4475acc63f6/f85c4218-0aef-4639-a0dc-11a66bf7298f"
 					(reference "R6")
-					(unit 1)
-				)
-			)
-		)
-	)
-	(symbol
-		(lib_id "Device:C")
-		(at 107.95 31.75 90)
-		(unit 1)
-		(body_style 1)
-		(exclude_from_sim no)
-		(in_bom yes)
-		(on_board yes)
-		(in_pos_files yes)
-		(dnp no)
-		(fields_autoplaced yes)
-		(property "Reference" "CBUS1"
-			(at 107.95 24.13 90)
-			(show_name no)
-			(do_not_autoplace no)
-			(effects
-				(font
-					(size 1.27 1.27)
-				)
-			)
-		)
-		(property "Value" "100nF"
-			(at 107.95 26.67 90)
-			(show_name no)
-			(do_not_autoplace no)
-			(effects
-				(font
-					(size 1.27 1.27)
-				)
-			)
-		)
-		(property "Footprint" "Package_TO_SOT_SMD:SOT-23-6"
-			(at 111.76 30.7848 0)
-			(hide yes)
-			(show_name no)
-			(do_not_autoplace no)
-			(effects
-				(font
-					(size 1.27 1.27)
-				)
-			)
-		)
-		(property "Datasheet" ""
-			(at 107.95 31.75 0)
-			(hide yes)
-			(show_name no)
-			(do_not_autoplace no)
-			(effects
-				(font
-					(size 1.27 1.27)
-				)
-			)
-		)
-		(property "Description" "Unpolarized capacitor"
-			(at 107.95 31.75 0)
-			(hide yes)
-			(show_name no)
-			(do_not_autoplace no)
-			(effects
-				(font
-					(size 1.27 1.27)
-				)
-			)
-		)
-		(pin "2"
-		)
-		(pin "1"
-		)
-		(instances
-			(project ""
-				(path "/83909f3c-09e4-4352-bc85-d5f4401c0e73"
-					(reference "CBUS")
-					(unit 1)
-				)
-			)
-			(project "DecodingBoard"
-				(path "/b438bce8-ca67-4245-91ae-f4475acc63f6/f85c4218-0aef-4639-a0dc-11a66bf7298f"
-					(reference "CBUS1")
 					(unit 1)
 				)
@@
 			)
 		)
-		(property "Footprint" ""
+		(property "Footprint" "Resistor_SMD:R_0402_1005Metric"
 			(at 73.66 38.608 90)
 			(hide yes)

Commit message: footprints updates
Parts:
- J3: footprint UJ20-C-H-G-SMT-1-P16-TR -> Footprints:SAMESKY_UJ20-C-H-G-SMT-1-P16-TR
Changed lines of the file:
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@@
 			)
 		)
-		(property "Footprint" "UJ20-C-H-G-SMT-1-P16-TR"
+		(property "Footprint" "Footprints:SAMESKY_UJ20-C-H-G-SMT-1-P16-TR"
 			(at 44.45 46.99 0)
 			(hide yes)

Commit message: First version of the layout
Parts:
- removed J3: USB_C_Receptacle_USB2.0_16P, Footprints:SAMESKY_UJ20-C-H-G-SMT-1-P16-TR, symbol Connector:USB_C_Receptacle_USB2.0_16P
- added J1: UJ20-C-H-G-SMT-1-P16-TR, Footprints:SAMESKY_UJ20-C-H-G-SMT-1-P16-TR, symbol UJ20-C-H-G-SMT-1-P16-TR:UJ20-C-H-G-SMT-1-P16-TR
Connections:
- net GND: now also J1.A1_B12 (GND), J1.B1_A12 (GND__1), J1.SH1 (SHIELD), J1.SH2 (SHIELD__1), J1.SH3 (SHIELD__2), J1.SH4 (SHIELD__3)
- net USB_CC1: now also J1.A5 (CC1)
- net USB_CC2: now also J1.B5 (CC2)
- net USB_D+: now also J1.A6 (DP1), J1.B6 (DP2)
- net USB_D-: now also J1.A7 (DN1), J1.B7 (DN2)
- net VBUS: now also J1.A4_B9 (VBUS), J1.B4_A9 (VBUS__1)
Other:
- note added: "USB-C"
- moved on the sheet: C31, R5, R6, U3
