File: Board V4/DecodingBoard/DecodingBoard.kicad_sch (KiCad schematic)
At the start: 22 parts, among them IC1 STM32WBA65CIU6, J1 Conn_01x03_Pin, J4 Conn_01x02_Pin, J5 Conn_01x06_Pin, SW1 TL3305BF100QG, SW2 TL3305BF100QG, U1 ESDS302DBVR

Commit message: update to the LDO footprint and C16 from 4.7 uF to 10 uF
Parts:
- renumbered XTALe to XTAL1
Connections:
- net STM32_power_supply_scheme/VDD renamed VDD_1
- net STM32_power_supply_scheme/VDD11 renamed VDD11
- net STM32_power_supply_scheme/VDDA renamed VDDA
- net STM32_power_supply_scheme/VDDANA renamed VDDANA
- net STM32_power_supply_scheme/VDDHPA renamed VDDHPA
- net STM32_power_supply_scheme/VDDRF renamed VDDRF
- net STM32_power_supply_scheme/VDDRPFA renamed VDDRFPA
- net STM32_power_supply_scheme/VDDSMPS renamed VDDSMPS
- net STM32_power_supply_scheme/VLXSMPS renamed VLXSMPS
- net STM32_power_supply_scheme/VSS renamed VSS
- net STM32_power_supply_scheme/VSSSMPS renamed VSSSMPS

Commit message: Addition of the BLE module and BOM
Parts:
- removed J1: Conn_01x03_Pin, Connector:Tag-Connect_TC2030-IDC-FP_2x03_P1.27mm_Vertical, symbol Connector:Conn_01x03_Pin
- removed J4: Conn_01x02_Pin, symbol Connector:Conn_01x02_Pin
- added J2: 2053380002, CONN_2053380000-SD_02_MOL, symbol 2053380002:2053380002
- added J4: 5040500491, CONN_5040500491_MOL, symbol 5040500491:5040500491
- C19, C20: footprint (none) -> Capacitor_SMD:C_0603_1608Metric
- C21, C22, C23: footprint (none) -> Capacitor_SMD:C_0402_1005Metric
- H1: footprint Module:Maple_Mini -> MountingHole:MountingHole_2.2mm_M2
- H2: footprint (none) -> MountingHole:MountingHole_2.2mm_M2
- J5: footprint (none) -> Connector_PinHeader_2.54mm:PinHeader_1x06_P2.54mm_Vertical_SMD_Pin1Left
- R1: footprint Package_DIP:DIP-8_W7.62mm -> Resistor_SMD:R_0402_1005Metric
- R14, R15, R16, R17, R2: footprint (none) -> Resistor_SMD:R_0402_1005Metric
Connections:
- net GND: now also J2.1, J4.3, J4.4
- net Power switching and voltage adaptation/VBat5V: now also J2.2
- net USART1_RX_CONN: now also J4.1
- net USART1_TX_CONN: now also J4.2
- net USART2_RX: now reaches IC1.14 (PD9)
- net USART2_TX: now reaches IC1.18 (PB8)
- net BLE Module/RF: no longer names the net of IC1.37 (RF)
- no-connect marks 25 -> 24
Other:
- sheet RF circuitry & antennas renamed BLE Module
- sheet BLE Module: file untitled.kicad_sch -> BLE Module.kicad_sch
- sheet BLE Module ports: added USART_RX_BLE, USART_TX_BLE, VCC; removed RF
- note added: "USART Connector with the prosthesis"
- moved on the sheet: J5

Commit message: footprints updates
Parts:
- IC1: footprint QFN50P700X700X60-49N-D -> Footprints:QFN50P700X700X60-49N-D
- J2: footprint CONN_2053380000-SD_02_MOL -> Footprints:CONN_2053380000-SD_02_MOL
- J4: footprint CONN_5040500491_MOL -> Footprints:CONN_5040500491_MOL
- SW1, SW2: footprint TL3305BF100QG:TL3305BF160QG -> Footprints:TL3305BF160QG
- U1: footprint DBV0005A_N -> Footprints:SOT95P280X145-5N
- XTAL1: footprint CX2016DB32000D0FLJCC:xtal4_CX2016DB_AVX -> Footprints:CX2016DB32000D0FLJCC
Changed lines of the file:
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@@
 			)
 		)
-		(property "Footprint" "TL3305BF100QG:TL3305BF160QG"
+		(property "Footprint" "Footprints:TL3305BF160QG"
 			(at 233.68 83.82 0)
 			(hide yes)
@@
 			)
 		)
-		(property "Footprint" "QFN50P700X700X60-49N-D"
+		(property "Footprint" "Footprints:QFN50P700X700X60-49N-D"
 			(at 171.45 171.12 0)
 			(hide yes)
@@
 			)
 		)
-		(property "Footprint" "TL3305BF100QG:TL3305BF160QG"
+		(property "Footprint" "Footprints:TL3305BF160QG"
 			(at 177.8 13.97 0)
 			(hide yes)
@@
 			)
 		)
-		(property "Footprint" "CONN_5040500491_MOL"
+		(property "Footprint" "Footprints:CONN_5040500491_MOL"
 			(at 39.37 85.09 0)
 			(hide yes)
@@
 			)
 		)
-		(property "Footprint" "DBV0005A_N"
+		(property "Footprint" "Footprints:SOT95P280X145-5N"
 			(at 48.26 107.95 0)
 			(hide yes)
@@
 			)
 		)
-		(property "Footprint" "CX2016DB32000D0FLJCC:xtal4_CX2016DB_AVX"
+		(property "Footprint" "Footprints:CX2016DB32000D0FLJCC"
 			(at 214.63 39.37 0)
 			(hide yes)
@@
 			)
 		)
-		(property "Footprint" "CONN_2053380000-SD_02_MOL"
+		(property "Footprint" "Footprints:CONN_2053380000-SD_02_MOL"
 			(at 55.88 182.88 0)
 			(hide yes)

Commit message: First version of the layout
Parts:
- H1, H2: footprint MountingHole:MountingHole_2.2mm_M2 -> MountingHole:MountingHole_2.2mm_M2_DIN965_Pad
Connections:
- net Power switching and voltage adaptation/VBat5V renamed Power
- net USART2_RX renamed USART2_RX_BLE
- net USART2_TX renamed USART2_RX_MCU
Other:
- moved on the sheet: H1, H2
Changed lines of the file:
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@@
 	)
 	(rectangle
+		(start 15.24 124.46)
+		(end 48.26 142.24)
+		(stroke
+			(width 0)
+			(type default)
+		)
+		(fill
+			(type none)
+		)
+	)
+	(rectangle
 		(start 19.05 41.91)
 		(end 49.53 62.23)
@@
 	)
 	(junction
-		(at 20.32 135.89)
+		(at 24.13 133.35)
 		(diameter 0)
 		(color 0 0 0 0)
@@
 	(wire
 		(pts
-			(xy 20.32 135.89) (xy 24.13 135.89)
+			(xy 24.13 133.35) (xy 27.94 133.35)
+		)
+		(stroke
+			(width 0)
+			(type default)
+		)
+	)
+	(wire
+		(pts
+			(xy 210.82 157.48) (xy 223.52 157.48)
 		)
 		(stroke
@@
 	(wire
 		(pts
-			(xy 20.32 142.24) (xy 24.13 142.24)
+			(xy 24.13 139.7) (xy 27.94 139.7)
 		)
 		(stroke
@@
 	(wire
 		(pts
-			(xy 20.32 135.89) (xy 20.32 142.24)
+			(xy 24.13 133.35) (xy 24.13 139.7)
+		)
+		(stroke
+			(width 0)
+			(type default)
+		)
+	)
+	(wire
+		(pts
+			(xy 208.28 153.67) (xy 223.52 153.67)
 		)
 		(stroke
@@
 	(wire
 		(pts
-			(xy 212.09 162.56) (xy 212.09 157.48)
+			(xy 210.82 162.56) (xy 210.82 157.48)
 		)
 		(stroke
@@
 	(wire
 		(pts
-			(xy 208.28 153.67) (xy 223.52 153.67)
-		)
-		(stroke
-			(width 0)
-			(type default)
-		)
-	)
-	(wire
-		(pts
 			(xy 261.62 46.99) (xy 266.7 46.99)
 		)
@@
 	(wire
 		(pts
-			(xy 139.7 162.56) (xy 212.09 162.56)
+			(xy 139.7 162.56) (xy 210.82 162.56)
 		)
 		(stroke
@@
 	(wire
 		(pts
-			(xy 24.13 135.89) (xy 24.13 133.35)
+			(xy 27.94 133.35) (xy 27.94 130.81)
 		)
 		(stroke
@@
 	(wire
 		(pts
-			(xy 212.09 157.48) (xy 223.52 157.48)
-		)
-		(stroke
-			(width 0)
-			(type default)
-		)
-	)
-	(wire
-		(pts
 			(xy 149.86 64.77) (xy 149.86 68.58)
 		)
@@
 	(wire
 		(pts
-			(xy 213.36 109.22) (xy 213.36 101.6)
+			(xy 20.32 133.35) (xy 24.13 133.35)
 		)
 		(stroke
@@
 	(wire
 		(pts
-			(xy 41.91 80.01) (xy 48.26 80.01)
+			(xy 213.36 109.22) (xy 213.36 101.6)
 		)
 		(stroke
@@
 	(wire
 		(pts
-			(xy 218.44 105.41) (xy 218.44 104.14)
+			(xy 41.91 80.01) (xy 48.26 80.01)
 		)
 		(stroke
@@
 	(wire
 		(pts
-			(xy 17.78 135.89) (xy 20.32 135.89)
+			(xy 218.44 105.41) (xy 218.44 104.14)
 		)
 		(stroke
@@
 		)
 	)
-	(label "USART2_TX"
-		(at 213.36 153.67 0)
+	(label "USART2_RX_BLE"
+		(at 210.82 157.48 0)
 		(effects
 			(font
@@
 		)
 	)
+	(label "USART2_RX_MCU"
+		(at 149.86 157.48 90)
+		(effects
+			(font
+				(size 1.016 1.016)
+			)
+			(justify left bottom)
+		)
+	)
 	(label "VDD_3"
 		(at 73.66 39.37 90)
@@
 		)
 	)
+	(label "USART2_TX_MCU"
+		(at 139.7 158.75 90)
+		(effects
+			(font
+				(size 1.016 1.016)
+			)
+			(justify left bottom)
+		)
+	)
 	(label "VDDANA"
 		(at 121.92 39.37 90)
@@
 		)
 	)
-	(label "USART2_RX"
-		(at 213.36 157.48 0)
+	(label "USART2_TX_BLE"
+		(at 210.82 153.67 0)
 		(effects
 			(font
@@
 		)
 	)
+	(label "Power"
+		(at 71.12 180.34 0)
+		(effects
+			(font
+				(size 1.016 1.016)
+			)
+			(justify left bottom)
+		)
+	)
 	(label "OSC_OUT"
 		(at 190.5 58.42 0)
@@
 	(symbol
 		(lib_id "power:GND")
-		(at 17.78 135.89 270)
+		(at 20.32 133.35 270)
 		(unit 1)
 		(body_style 1)
@@
 		(dnp no)
 		(property "Reference" "#PWR045"
-			(at 11.43 135.89 0)
+			(at 13.97 133.35 0)
 			(hide yes)
 			(show_name no)
@@
 		)
 		(property "Value" "GND"
-			(at 18.542 138.938 90)
+			(at 21.082 136.398 90)
 			(show_name no)
 			(do_not_autoplace no)
@@
 		)
 		(property "Footprint" ""
-			(at 17.78 135.89 0)
+			(at 20.32 133.35 0)
 			(hide yes)
 			(show_name no)
@@
 		)
 		(property "Datasheet" ""
-			(at 17.78 135.89 0)
+			(at 20.32 133.35 0)
 			(hide yes)
 			(show_name no)
@@
 		)
 		(property "Description" "Power symbol creates a global label with name \"GND\" , ground"
-			(at 17.78 135.89 0)
+			(at 20.32 133.35 0)
 			(hide yes)
 			(show_name no)
@@
 	(symbol
 		(lib_id "Mechanical:MountingHole_Pad")
-		(at 24.13 130.81 0)
+		(at 27.94 128.27 0)
 		(unit 1)
 		(body_style 1)
@@
 		(fields_autoplaced yes)
 		(property "Reference" "H1"
-			(at 26.67 128.2699 0)
+			(at 30.48 125.7299 0)
 			(show_name no)
 			(do_not_autoplace no)
@@
 		)
 		(property "Value" "MountingHole_Pad"
-			(at 26.67 130.8099 0)
+			(at 30.48 128.2699 0)
 			(show_name no)
 			(do_not_autoplace no)
@@
 			)
 		)
-		(property "Footprint" "MountingHole:MountingHole_2.2mm_M2"
-			(at 24.13 130.81 0)
+		(property "Footprint" "MountingHole:MountingHole_2.2mm_M2_DIN965_Pad"
+			(at 27.94 128.27 0)
 			(hide yes)
 			(show_name no)
@@
 		)
 		(property "Datasheet" ""
-			(at 24.13 130.81 0)
+			(at 27.94 128.27 0)
 			(hide yes)
 			(show_name no)
@@
 		)
 		(property "Description" "Mounting Hole with connection"
-			(at 24.13 130.81 0)
+			(at 27.94 128.27 0)
 			(hide yes)
 			(show_name no)
@@
 	(symbol
 		(lib_id "Mechanical:MountingHole_Pad")
-		(at 24.13 139.7 0)
+		(at 27.94 137.16 0)
 		(unit 1)
 		(body_style 1)
@@
 		(fields_autoplaced yes)
 		(property "Reference" "H2"
-			(at 26.67 137.1599 0)
+			(at 30.48 134.6199 0)
 			(show_name no)
 			(do_not_autoplace no)
@@
 		)
 		(property "Value" "MountingHole_Pad"
-			(at 26.67 139.6999 0)
+			(at 30.48 137.1599 0)
 			(show_name no)
 			(do_not_autoplace no)
@@
 			)
 		)
-		(property "Footprint" "MountingHole:MountingHole_2.2mm_M2"
-			(at 24.13 139.7 0)
+		(property "Footprint" "MountingHole:MountingHole_2.2mm_M2_DIN965_Pad"
+			(at 27.94 137.16 0)
 			(hide yes)
 			(show_name no)
@@
 		)
 		(property "Datasheet" ""
-			(at 24.13 139.7 0)
+			(at 27.94 137.16 0)
 			(hide yes)
 			(show_name no)
@@
 		)
 		(property "Description" "Mounting Hole with connection"
-			(at 24.13 139.7 0)
+			(at 27.94 137.16 0)
 			(hide yes)
 			(show_name no)
@@
 		)
 		(pin "USART_RX_BLE" input
-			(at 223.52 153.67 180)
+			(at 223.52 157.48 180)
 			(effects
 				(font
@@
 		)
 		(pin "USART_TX_BLE" input
-			(at 223.52 157.48 180)
+			(at 223.52 153.67 180)
 			(effects
 				(font

Commit message: progress on the layout
Parts:
- removed J2: 2053380002, Footprints:CONN_2053380000-SD_02_MOL, symbol 2053380002:2053380002
- removed J4: 5040500491, Footprints:CONN_5040500491_MOL, symbol 5040500491:5040500491
- removed J5: Conn_01x06_Pin, Connector_PinHeader_2.54mm:PinHeader_1x06_P2.54mm_Vertical_SMD_Pin1Left, symbol Connector:Conn_01x06_Pin
- added J3: TSM-106-02-T-SH-LC, Footprints:SAMTEC_TSM-106-02-T-SH-LC, symbol TSM-106-02-T-SH-LC:TSM-106-02-T-SH-LC
- added J4: 2053380004, Footprints:CONN_2053380000-SD_02_MOL, symbol 2053380002_4pins:2053380004
- added J6: 5040500691, Footprints:CONN_5040500491_MOL, symbol 5040500691_6pins:5040500691
Connections:
- net +3.3V: now also J3.01
- net GND: now also J3.02, J4.1, J4.3, J4.4, J6.3, J6.4, J6.5, J6.6
- net Power: now also J4.2
- net SWDCLK: now also J3.04
- net SWDIO: now also J3.05
- net SWD_NRST: now also J3.03
- net SWD_TRACES: now also J3.06
- net USART1_RX_CONN: now also J6.1
- net USART1_TX_CONN: now also J6.2
